Commit message: Add moveit assistant fixes

File: config/gazebo_wp_manipulator.urdf (robot description, URDF)
Before this commit: robot wp_manipulator, 8 links, 7 joints
Links:
- removed link base
- removed link end_effector_base
- removed link link1
- removed link link2
- removed link link3
- removed link link4
- removed link link5
Joints:
- removed joint joint1
- removed joint joint2
- removed joint joint3
- removed joint joint4
- removed joint joint5
- removed joint jointEndEffectorBase
- removed joint wp_base_joint
